Commit message: Basic Work Cell Setting with Motion Planning

File: src/my_ur_description/urdf/ur_system.xacro (robot description, xacro)
@@ -6,27 +6,58 @@
   <link name="easydesk">
     <visual>
-      <geometry><box size="1.5 1.0 0.05"/></geometry>
+      <geometry><box size="1.2 0.8 0.05"/></geometry>
       <material name="light_grey"><color rgba="0.7 0.7 0.7 1"/></material>
     </visual>
     <collision>
-      <geometry><box size="1.5 1.0 0.05"/></geometry>
+      <geometry><box size="1.2 0.8 0.05"/></geometry>
     </collision>
   </link>
   <joint name="world_to_desk" type="fixed">
     <parent link="world"/><child link="easydesk"/>
-    <origin xyz="0 0 0.75" rpy="0 0 0"/>
+    <origin xyz="0.7 0 0.9" rpy="0 0 0"/>
   </joint>
-  <link name="safety_wall">
-    <collision>
-      <geometry><box size="1.5 0.05 2.0"/></geometry>
-    </collision>
+  <link name="back_wall">
+    <collision><geometry><box size="2.5 0.01 1.5"/></geometry></collision>
     <visual>
-      <geometry><box size="1.5 0.01 2.0"/></geometry>
-      <material name="transparent_red"><color rgba="1 0 0 0.2"/></material>
+      <geometry><box size="2.5 0.01 1.5"/></geometry>
+      <material name="transparent_red"><color rgba="1 0 0 0.05"/></material>
     </visual>
   </link>
-  <joint name="desk_to_wall" type="fixed">
-    <parent link="easydesk"/><child link="safety_wall"/>
-    <origin xyz="0 0.5 1.0" rpy="0 0 0"/>
+  <joint name="desk_to_back_wall" type="fixed">
+    <parent link="easydesk"/><child link="back_wall"/>
+    <origin xyz="-0.25 0.6 0.75" rpy="0 0 0"/>
+  </joint>
+  <link name="front_wall">
+    <collision><geometry><box size="2.5 0.01 1.5"/></geometry></collision>
+    <visual>
+      <geometry><box size="2.5 0.01 1.5"/></geometry>
+      <material name="transparent_red"><color rgba="1 0 0 0.05"/></material>
+    </visual>
+  </link>
+  <joint name="desk_to_front_wall" type="fixed">
+    <parent link="easydesk"/><child link="front_wall"/>
+    <origin xyz="-0.25 -0.45 0.75" rpy="0 0 0"/>
+  </joint>
+  <link name="left_wall">
+    <collision><geometry><box size="0.01 1.2 1.5"/></geometry></collision>
+    <visual>
+      <geometry><box size="0.01 1.2 1.5"/></geometry>
+      <material name="transparent_red"><color rgba="1 0 0 0.05"/></material>
+    </visual>
+  </link>
+  <joint name="desk_to_left_wall" type="fixed">
+    <parent link="easydesk"/><child link="left_wall"/>
+    <origin xyz="-1.0 0 0.75" rpy="0 0 0"/>
+  </joint>
+  <link name="right_wall">
+    <collision><geometry><box size="0.01 1.2 1.5"/></geometry></collision>
+    <visual>
+      <geometry><box size="0.01 1.2 1.5"/></geometry>
+      <material name="transparent_red"><color rgba="1 0 0 0.05"/></material>
+    </visual>
+  </link>
+  <joint name="desk_to_right_wall" type="fixed">
+    <parent link="easydesk"/><child link="right_wall"/>
+    <origin xyz="0.7 0 0.75" rpy="0 0 0"/>
   </joint>
   <xacro:macro name="d435_mount" params="prefix x y z yaw">
@@ -36,4 +67,7 @@
         <material name="blue"><color rgba="0 0 1 1"/></material>
       </visual>
+      <collision>
+        <geometry><box size="0.09 0.025 0.025"/></geometry>
+      </collision>
     </link>
     <joint name="desk_to_${prefix}_cam" type="fixed">
@@ -42,7 +76,7 @@
     </joint>
   </xacro:macro>
-  <xacro:d435_mount prefix="cam_left" x="-0.6" y="-0.4" z="0.4" yaw="0.78"/>
-  <xacro:d435_mount prefix="cam_right" x="0.6" y="-0.4" z="0.4" yaw="2.35"/>
-<xacro:ur_robot name="ur" tf_prefix="" parent="easydesk"
+  <xacro:d435_mount prefix="cam_left" x="0.2" y="-0.4" z="0.2" yaw="1.57"/>
+  <xacro:d435_mount prefix="cam_right" x="0.6" y="-0.0" z="0.4" yaw="3.14"/>
+  <xacro:ur_robot name="ur" tf_prefix="" parent="easydesk"
     joint_limits_parameters_file="$(find ur_description)/config/ur12e/joint_limits.yaml"
     kinematics_parameters_file="$(find ur_description)/config/ur12e/default_kinematics.yaml"
@@ -51,27 +85,23 @@
     use_fake_hardware="true"
     fake_sensor_commands="true" >
-    <origin xyz="0 0 0.025" rpy="0 0 0" />
+    <origin xyz="-0.7 0 0.025" rpy="0 0 0" />
   </xacro:ur_robot>
-<xacro:robotiq_gripper name="robotiq_85" prefix="" parent="tool0" include_ros2_control="false">
+  <xacro:robotiq_gripper name="robotiq_85" prefix="" parent="tool0" include_ros2_control="false">
     <origin xyz="0 0 0" rpy="0 0 0" />
   </xacro:robotiq_gripper>
-<ros2_control name="RobotiqGripperHardwareInterface" type="system">
-  <hardware>
-    <plugin>mock_components/GenericSystem</plugin>
-  </hardware>
-  <joint name="robotiq_85_left_knuckle_joint">
-    <command_interface name="position"/>
-    <state_interface name="position">
-      <param name="initial_value">0.0</param>
-    </state_interface>
-    <state_interface name="velocity">
-      <param name="initial_value">0.0</param>
-    </state_interface>
-  </joint>
-  <joint name="robotiq_85_right_knuckle_joint"><state_interface name="position"/></joint>
-  <joint name="robotiq_85_left_inner_knuckle_joint"><state_interface name="position"/></joint>
-  <joint name="robotiq_85_right_inner_knuckle_joint"><state_interface name="position"/></joint>
-  <joint name="robotiq_85_left_finger_tip_joint"><state_interface name="position"/></joint>
-  <joint name="robotiq_85_right_finger_tip_joint"><state_interface name="position"/></joint>
-</ros2_control>
+  <ros2_control name="RobotiqGripperHardwareInterface" type="system">
+    <hardware>
+      <plugin>mock_components/GenericSystem</plugin>
+    </hardware>
+    <joint name="robotiq_85_left_knuckle_joint">
+      <command_interface name="position"/>
+      <state_interface name="position"><param name="initial_value">0.0</param></state_interface>
+      <state_interface name="velocity"><param name="initial_value">0.0</param></state_interface>
+    </joint>
+    <joint name="robotiq_85_right_knuckle_joint"><param name="mimic">robotiq_85_left_knuckle_joint</param><param name="multiplier">-1.0</param><command_interface name="position"/><state_interface name="position"/></joint>
+    <joint name="robotiq_85_left_inner_knuckle_joint"><param name="mimic">robotiq_85_left_knuckle_joint</param><param name="multiplier">1.0</param><command_interface name="position"/><state_interface name="position"/></joint>
+    <joint name="robotiq_85_right_inner_knuckle_joint"><param name="mimic">robotiq_85_left_knuckle_joint</param><param name="multiplier">-1.0</param><command_interface name="position"/><state_interface name="position"/></joint>
+    <joint name="robotiq_85_left_finger_tip_joint"><param name="mimic">robotiq_85_left_knuckle_joint</param><param name="multiplier">-1.0</param><command_interface name="position"/><state_interface name="position"/></joint>
+    <joint name="robotiq_85_right_finger_tip_joint"><param name="mimic">robotiq_85_left_knuckle_joint</param><param name="multiplier">1.0</param><command_interface name="position"/><state_interface name="position"/></joint>
+  </ros2_control>
 </robot>

Commit message: Intel Depth Cameras D435 Realistic Added

File: src/my_ur_description/urdf/ur_system.xacro (robot description, xacro)
@@ -64,8 +64,11 @@
     <link name="${prefix}_camera_link">
       <visual>
-        <geometry><box size="0.09 0.025 0.025"/></geometry>
-        <material name="blue"><color rgba="0 0 1 1"/></material>
+        <origin xyz="0 0 0" rpy="${pi/2} 0 ${pi/2}"/>
+        <geometry>
+          <mesh filename="package://realsense2_description/meshes/d435.dae" />
+        </geometry>
       </visual>
       <collision>
+        <origin xyz="0 0 0" rpy="${pi/2} 0 ${pi/2}"/>
         <geometry><box size="0.09 0.025 0.025"/></geometry>
       </collision>
@@ -74,4 +77,10 @@
       <parent link="easydesk"/><child link="${prefix}_camera_link"/>
       <origin xyz="${x} ${y} ${z}" rpy="0 0.5 ${yaw}"/>
+    </joint>
+    <link name="${prefix}_camera_optical_frame"/>
+    <joint name="${prefix}_optical_joint" type="fixed">
+      <parent link="${prefix}_camera_link"/>
+      <child link="${prefix}_camera_optical_frame"/>
+      <origin xyz="0 0 0" rpy="${-pi/2} 0 ${-pi/2}"/>
     </joint>
   </xacro:macro>

Commit message: Save current state before reverting to stabel fake sim

File: src/my_ur_description/urdf/ur_system.xacro (robot description, xacro)
@@ -1,4 +1,6 @@
 <?xml version="1.0"?>
-<robot xmlns:xacro="http://wiki.ros.org/xacro" name="ur12e_system">
+<robot xmlns:xacro="http://wiki.ros.org/xacro" name="ur">
+  <xacro:arg name="use_fake_hardware" default="false" />
+  <xacro:arg name="external_interface_adapter" default="false" />
   <xacro:include filename="$(find ur_description)/urdf/ur_macro.xacro"/>
   <xacro:include filename="$(find robotiq_description)/urdf/robotiq_2f_85_macro.urdf.xacro"/>
@@ -88,11 +90,10 @@
   <xacro:d435_mount prefix="cam_right" x="0.6" y="-0.0" z="0.4" yaw="3.14"/>
   <xacro:ur_robot name="ur" tf_prefix="" parent="easydesk"
-    joint_limits_parameters_file="$(find ur_description)/config/ur12e/joint_limits.yaml"
-    kinematics_parameters_file="$(find ur_description)/config/ur12e/default_kinematics.yaml"
-    physical_parameters_file="$(find ur_description)/config/ur12e/physical_parameters.yaml"
-    visual_parameters_file="$(find ur_description)/config/ur12e/visual_parameters.yaml"
-    use_fake_hardware="true"
-    fake_sensor_commands="true" >
-    <origin xyz="-0.7 0 0.025" rpy="0 0 0" />
+    joint_limits_parameters_file="$(find ur_description)/config/ur10e/joint_limits.yaml"
+    kinematics_parameters_file="$(find ur_description)/config/ur10e/default_kinematics.yaml"
+    physical_parameters_file="$(find ur_description)/config/ur10e/physical_parameters.yaml"
+    visual_parameters_file="$(find ur_description)/config/ur10e/visual_parameters.yaml"
+    >
+    <origin xyz="-0.8 0 -0.05" rpy="0 0 0" />
   </xacro:ur_robot>
   <xacro:robotiq_gripper name="robotiq_85" prefix="" parent="tool0" include_ros2_control="false">
